File: TSAL_HV_PCB.kicad_sch (KiCad schematic)
At the start: 36 parts, among them J3 Conn_01x03_Socket, J4 Conn_01x03_Socket, K1 SPU01M-12, U1 LM393, U2 4N35, U3 TPS7B88-Q1

Commit message: Fixed 3d model paths
Parts:
- J3, J4: footprint MyLibrary:MolexMicrofitPlus1x3 -> yfs:MolexMicrofitPlus1x3
- K1: footprint MyLibrary:SPU01M-12 -> yfs:SPU01M-12
Changed lines of the file:
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@@
 			)
 		)
-		(property "Footprint" "MyLibrary:MolexMicrofitPlus1x3"
+		(property "Footprint" "yfs:MolexMicrofitPlus1x3"
 			(at 247.65 69.85 0)
 			(effects
@@
 			)
 		)
-		(property "Footprint" "MyLibrary:MolexMicrofitPlus1x3"
+		(property "Footprint" "yfs:MolexMicrofitPlus1x3"
 			(at 39.37 38.1 0)
 			(effects
@@
 			)
 		)
-		(property "Footprint" "MyLibrary:SPU01M-12"
+		(property "Footprint" "yfs:SPU01M-12"
 			(at 137.16 38.1 0)
 			(effects
